File: electronics/lft_keyboard.kicad_sch (KiCad schematic)
At the start: 0 parts

Commit message: add io expander and switches to schem
Parts:
- added SW1, SW10, SW11, SW12, SW13, SW14, SW15, SW16, SW17, SW18, SW19, SW2, SW20, SW21, SW22, SW23, SW24, SW25, SW26, SW27, SW28, SW29, SW3, SW4, SW5, SW6, SW7, SW8, SW9: SW_SPST, Kailh:Kailh_socket_MX, symbol Kailh:SW_SPST
- added U2: PCA9506DGG, PCA9506:PCA9506DGG, symbol PCA9506:PCA9506DGG
