File: electronics/rgt_keyboard.kicad_sch (KiCad schematic)
At the start: 0 parts

Commit message: add io expander and switches to schem
Parts:
- added SW30, SW31, SW32, SW33, SW34, SW35, SW36, SW37, SW38, SW39, SW40, SW41, SW42, SW43, SW44, SW45, SW46, SW47, SW48, SW49, SW50, SW51, SW52, SW53, SW54, SW55, SW56, SW57, SW58: SW_SPST, Kailh:Kailh_socket_MX, symbol Kailh:SW_SPST
- added U3: PCA9506DGG, PCA9506:PCA9506DGG, symbol PCA9506:PCA9506DGG
