File: electronics/arrw_macro.kicad_sch (KiCad schematic)
At the start: 0 parts

Commit message: add io expander and switches to schem
Parts:
- added SW59, SW60, SW61, SW62, SW63, SW64, SW65, SW66, SW67, SW68: SW_SPST, Kailh:Kailh_socket_MX, symbol Kailh:SW_SPST
- added U4: MAX7314AEG+, MAX7314AEG:MAX7314AEG&plus_, symbol MAX7314AEG:MAX7314AEG+
Changed lines of the file:
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@@
     (company "OSHMount Tech")
   )
+  (symbol (lib_id "Kailh:SW_SPST") (at 81.28 170.18 0) (unit 1)
+    (in_bom yes) (on_board yes) (fields_autoplaced)
+    (property "Reference" "SW68" (id 0) (at 81.28 163.83 0))
+    (property "Value" "SW_SPST" (id 1) (at 81.28 166.37 0))
+    (property "Footprint" "Kailh:Kailh_socket_MX" (id 2) (at 81.28 170.18 0)
+      (effects (font (size 1.27 1.27)) hide)
+    )
+    (property "Datasheet" "${KIPRJMOD}/lib/Kailh/Kailh_Polia_datasheet.pdf" (id 3) (at 81.28 170.18 0)
+      (effects (font (size 1.27 1.27)) hide)
+    )
+    (pin "1")
+    (pin "2")
+  )
+  (symbol (lib_id "Kailh:SW_SPST") (at 40.64 170.18 0) (unit 1)
+    (in_bom yes) (on_board yes) (fields_autoplaced)
+    (property "Reference" "SW66" (id 0) (at 40.64 163.83 0))
+    (property "Value" "SW_SPST" (id 1) (at 40.64 166.37 0))
+    (property "Footprint" "Kailh:Kailh_socket_MX" (id 2) (at 40.64 170.18 0)
+      (effects (font (size 1.27 1.27)) hide)
+    )
+    (property "Datasheet" "${KIPRJMOD}/lib/Kailh/Kailh_Polia_datasheet.pdf" (id 3) (at 40.64 170.18 0)
+      (effects (font (size 1.27 1.27)) hide)
+    )
+    (pin "1")
+    (pin "2")
+  )
+  (symbol (lib_id "Kailh:SW_SPST") (at 60.96 170.18 0) (unit 1)
+    (in_bom yes) (on_board yes) (fields_autoplaced)
+    (property "Reference" "SW67" (id 0) (at 60.96 163.83 0))
+    (property "Value" "SW_SPST" (id 1) (at 60.96 166.37 0))
+    (property "Footprint" "Kailh:Kailh_socket_MX" (id 2) (at 60.96 170.18 0)
+      (effects (font (size 1.27 1.27)) hide)
+    )
+    (property "Datasheet" "${KIPRJMOD}/lib/Kailh/Kailh_Polia_datasheet.pdf" (id 3) (at 60.96 170.18 0)
+      (effects (font (size 1.27 1.27)) hide)
+    )
+    (pin "1")
+    (pin "2")
+  )
+  (symbol (lib_id "Kailh:SW_SPST") (at 81.28 106.68 0) (unit 1)
+    (in_bom yes) (on_board yes) (fields_autoplaced)
+    (property "Reference" "SW61" (id 0) (at 81.28 100.33 0))
+    (property "Value" "SW_SPST" (id 1) (at 81.28 102.87 0))
+    (property "Footprint" "Kailh:Kailh_socket_MX" (id 2) (at 81.28 106.68 0)
+      (effects (font (size 1.27 1.27)) hide)
+    )
+    (property "Datasheet" "${KIPRJMOD}/lib/Kailh/Kailh_Polia_datasheet.pdf" (id 3) (at 81.28 106.68 0)
+      (effects (font (size 1.27 1.27)) hide)
+    )
+    (pin "1")
+    (pin "2")
+  )
+  (symbol (lib_id "Kailh:SW_SPST") (at 60.96 154.94 0) (unit 1)
+    (in_bom yes) (on_board yes) (fields_autoplaced)
+    (property "Reference" "SW65" (id 0) (at 60.96 148.59 0))
+    (property "Value" "SW_SPST" (id 1) (at 60.96 151.13 0))
+    (property "Footprint" "Kailh:Kailh_socket_MX" (id 2) (at 60.96 154.94 0)
+      (effects (font (size 1.27 1.27)) hide)
+    )
+    (property "Datasheet" "${KIPRJMOD}/lib/Kailh/Kailh_Polia_datasheet.pdf" (id 3) (at 60.96 154.94 0)
+      (effects (font (size 1.27 1.27)) hide)
+    )
+    (pin "1")
+    (pin "2")
+  )
+  (symbol (lib_id "MAX7314AEG:MAX7314AEG+") (at 52.07 46.99 0) (unit 1)
+    (in_bom yes) (on_board yes) (fields_autoplaced)
+    (property "Reference" "U4" (id 0) (at 87.63 35.56 0)
+      (effects (font (size 1.524 1.524)))
+    )
+    (property "Value" "MAX7314AEG+" (id 1) (at 87.63 39.37 0)
+      (effects (font (size 1.524 1.524)))
+    )
+    (property "Footprint" "MAX7314AEG:MAX7314AEG&plus_" (id 2) (at 87.63 40.894 0)
+      (effects (font (size 1.524 1.524)) hide)
+    )
+    (property "Datasheet" "${KIPRJMOD}/lib/MAX7314AEG/MAX7314AEG+.pdf" (id 3) (at 52.07 46.99 0)
+      (effects (font (size 1.524 1.524)) hide)
+    )
+    (pin "1")
+    (pin "10")
+    (pin "11")
+    (pin "12")
+    (pin "13")
+    (pin "14")
+    (pin "15")
+    (pin "16")
+    (pin "17")
+    (pin "18")
+    (pin "19")
+    (pin "2")
+    (pin "20")
+    (pin "21")
+    (pin "22")
+    (pin "23")
+    (pin "24")
+    (pin "3")
+    (pin "4")
+    (pin "5")
+    (pin "6")
+    (pin "7")
+    (pin "8")
+    (pin "9")
+  )
+  (symbol (lib_id "Kailh:SW_SPST") (at 60.96 106.68 0) (unit 1)
+    (in_bom yes) (on_board yes) (fields_autoplaced)
+    (property "Reference" "SW60" (id 0) (at 60.96 100.33 0))
+    (property "Value" "SW_SPST" (id 1) (at 60.96 102.87 0))
+    (property "Footprint" "Kailh:Kailh_socket_MX" (id 2) (at 60.96 106.68 0)
+      (effects (font (size 1.27 1.27)) hide)
+    )
+    (property "Datasheet" "${KIPRJMOD}/lib/Kailh/Kailh_Polia_datasheet.pdf" (id 3) (at 60.96 106.68 0)
+      (effects (font (size 1.27 1.27)) hide)
+    )
+    (pin "1")
+    (pin "2")
+  )
+  (symbol (lib_id "Kailh:SW_SPST") (at 40.64 121.92 0) (unit 1)
+    (in_bom yes) (on_board yes) (fields_autoplaced)
+    (property "Reference" "SW62" (id 0) (at 40.64 115.57 0))
+    (property "Value" "SW_SPST" (id 1) (at 40.64 118.11 0))
+    (property "Footprint" "Kailh:Kailh_socket_MX" (id 2) (at 40.64 121.92 0)
+      (effects (font (size 1.27 1.27)) hide)
+    )
+    (property "Datasheet" "${KIPRJMOD}/lib/Kailh/Kailh_Polia_datasheet.pdf" (id 3) (at 40.64 121.92 0)
+      (effects (font (size 1.27 1.27)) hide)
+    )
+    (pin "1")
+    (pin "2")
+  )
+  (symbol (lib_id "Kailh:SW_SPST") (at 40.64 106.68 0) (unit 1)
+    (in_bom yes) (on_board yes) (fields_autoplaced)
+    (property "Reference" "SW59" (id 0) (at 40.64 100.33 0))
+    (property "Value" "SW_SPST" (id 1) (at 40.64 102.87 0))
+    (property "Footprint" "Kailh:Kailh_socket_MX" (id 2) (at 40.64 106.68 0)
+      (effects (font (size 1.27 1.27)) hide)
+    )
+    (property "Datasheet" "${KIPRJMOD}/lib/Kailh/Kailh_Polia_datasheet.pdf" (id 3) (at 40.64 106.68 0)
+      (effects (font (size 1.27 1.27)) hide)
+    )
+    (pin "1")
+    (pin "2")
+  )
+  (symbol (lib_id "Kailh:SW_SPST") (at 60.96 121.92 0) (unit 1)
+    (in_bom yes) (on_board yes) (fields_autoplaced)
+    (property "Reference" "SW63" (id 0) (at 60.96 115.57 0))
+    (property "Value" "SW_SPST" (id 1) (at 60.96 118.11 0))
+    (property "Footprint" "Kailh:Kailh_socket_MX" (id 2) (at 60.96 121.92 0)
+      (effects (font (size 1.27 1.27)) hide)
+    )
+    (property "Datasheet" "${KIPRJMOD}/lib/Kailh/Kailh_Polia_datasheet.pdf" (id 3) (at 60.96 121.92 0)
+      (effects (font (size 1.27 1.27)) hide)
+    )
+    (pin "1")
+    (pin "2")
+  )
+  (symbol (lib_id "Kailh:SW_SPST") (at 81.28 121.92 0) (unit 1)
+    (in_bom yes) (on_board yes) (fields_autoplaced)
+    (property "Reference" "SW64" (id 0) (at 81.28 115.57 0))
+    (property "Value" "SW_SPST" (id 1) (at 81.28 118.11 0))
+    (property "Footprint" "Kailh:Kailh_socket_MX" (id 2) (at 81.28 121.92 0)
+      (effects (font (size 1.27 1.27)) hide)
+    )
+    (property "Datasheet" "${KIPRJMOD}/lib/Kailh/Kailh_Polia_datasheet.pdf" (id 3) (at 81.28 121.92 0)
+      (effects (font (size 1.27 1.27)) hide)
+    )
+    (pin "1")
+    (pin "2")
+  )
 )
