File: electronics/num_pad.kicad_sch (KiCad schematic)
At the start: 0 parts

Commit message: add io expander and switches to schem
Parts:
- added SW69, SW70, SW71, SW72, SW73, SW74, SW75, SW76, SW77, SW78, SW79, SW80, SW81, SW82, SW83, SW84, SW85: SW_SPST, Kailh:Kailh_socket_MX, symbol Kailh:SW_SPST
- added U5: MAX7314AEG+, MAX7314AEG:MAX7314AEG&plus_, symbol MAX7314AEG:MAX7314AEG+
